File: hw/kicad/bttoy.sch (KiCad schematic (older format))
At the start: 0 parts

Commit message: - start basic schematic, few ic's
Parts:
- added J?: USB-micro-b, symbol USB-micro-b
- added U?: MKL05Z32VLC4, symbol MKL05Z32VLC4
- added U?: MCP73831, symbol MCP73831
- added U?: AAT3221/MIC5504, symbol AAT3221
Changed lines of the file:
@@
 LIBS:contrib
 LIBS:valves
+LIBS:kicadlib
+LIBS:bttoy-cache
 EELAYER 25 0
 EELAYER END
@@
 Comment4 ""
 $EndDescr
+$Comp
+L MKL05Z32VLC4 U?
+U 1 1 54977F03
+P 4250 3450
+F 0 "U?" H 4650 3650 60  0000 C CNN
+F 1 "MKL05Z32VLC4" H 4700 3500 60  0000 C CNN
+F 2 "" H 4250 3450 60  0000 C CNN
+F 3 "" H 4250 3450 60  0000 C CNN
+	1    4250 3450
+	1    0    0    -1
+$EndComp
+$Comp
+L MCP73831 U?
+U 1 1 54977F63
+P 3600 6000
+F 0 "U?" H 3600 5700 60  0000 C CNN
+F 1 "MCP73831" H 3600 6300 60  0000 C CNN
+F 2 "" H 3600 6000 60  0000 C CNN
+F 3 "" H 3600 6000 60  0000 C CNN
+	1    3600 6000
+	1    0    0    -1
+$EndComp
+$Comp
+L USB-micro-b J?
+U 1 1 5497803A
+P 2100 3550
+F 0 "J?" H 2100 2950 60  0000 C CNN
+F 1 "USB-micro-b" H 2100 4200 60  0000 C CNN
+F 2 "" H 2100 3550 60  0000 C CNN
+F 3 "" H 2100 3550 60  0000 C CNN
+	1    2100 3550
+	1    0    0    -1
+$EndComp
+$Comp
+L AAT3221 U?
+U 1 1 5497812B
+P 5300 5850
+F 0 "U?" H 5300 5650 60  0000 C CNN
+F 1 "AAT3221/MIC5504" H 5300 6250 60  0000 C CNN
+F 2 "" H 5300 5850 60  0000 C CNN
+F 3 "" H 5300 5850 60  0000 C CNN
+	1    5300 5850
+	1    0    0    -1
+$EndComp
 $EndSCHEMATC
