File: hw/kicad/bttoy.sch (KiCad schematic (older format))
At the start: 46 parts, among them J1 USB-micro-b, J2 HC-07_BLUETOOTH, J3 ARM_10PIN, P1 gnd, P10 M1+, P11 M1-, P12 M2+, P13 M2-, P14 B-, P15 B+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

Commit message: gerbers and done
Parts:
- P1, P16: value gnd -> g
- P2: value i2c_sda -> sd
- P3: value i2c_scl -> sc
- P4: value spi_ss -> cs
- P5: value spi_miso -> mi
- P6: value spi_mosi -> mo
- P7: value spi_clk -> ck
Connections:
- net acc_spi_miso is gone; now on net spi_miso: U4.10 (PTA6)
- net mps_en: now also U4.17 (PTB1)
- no-connect marks 46 -> 45
Changed lines of the file:
@@
 spi_mosi
 Text Label 6150 3150 3    60   ~ 0
-acc_spi_miso
+spi_miso
 Text Label 7050 3150 3    60   ~ 0
 spi_sclk
@@
 P 5600 6150
 F 0 "P6" H 5600 6450 40  0000 C CNN
-F 1 "spi_mosi" H 5600 6400 30  0000 C CNN
+F 1 "mo" H 5600 6400 30  0000 C CNN
 F 2 "kicadlib:TEST_0.100" H 5600 6150 60  0001 C CNN
 F 3 "" H 5600 6150 60  0000 C CNN
@@
 P 5400 6150
 F 0 "P5" H 5400 6450 40  0000 C CNN
-F 1 "spi_miso" H 5400 6400 30  0000 C CNN
+F 1 "mi" H 5400 6400 30  0000 C CNN
 F 2 "kicadlib:TEST_0.100" H 5400 6150 60  0001 C CNN
 F 3 "" H 5400 6150 60  0000 C CNN
@@
 P 5200 6150
 F 0 "P4" H 5200 6450 40  0000 C CNN
-F 1 "spi_ss" H 5200 6400 30  0000 C CNN
+F 1 "cs" H 5200 6400 30  0000 C CNN
 F 2 "kicadlib:TEST_0.100" H 5200 6150 60  0001 C CNN
 F 3 "" H 5200 6150 60  0000 C CNN
@@
 P 5800 6150
 F 0 "P7" H 5800 6450 40  0000 C CNN
-F 1 "spi_clk" H 5800 6400 30  0000 C CNN
+F 1 "ck" H 5800 6400 30  0000 C CNN
 F 2 "kicadlib:TEST_0.100" H 5800 6150 60  0001 C CNN
 F 3 "" H 5800 6150 60  0000 C CNN
@@
 P 4500 6150
 F 0 "P2" H 4500 6450 40  0000 C CNN
-F 1 "i2c_sda" H 4500 6400 30  0000 C CNN
+F 1 "sd" H 4500 6400 30  0000 C CNN
 F 2 "kicadlib:TEST_0.100" H 4500 6150 60  0001 C CNN
 F 3 "" H 4500 6150 60  0000 C CNN
@@
 P 4700 6150
 F 0 "P3" H 4700 6450 40  0000 C CNN
-F 1 "i2c_scl" H 4700 6400 30  0000 C CNN
+F 1 "sc" H 4700 6400 30  0000 C CNN
 F 2 "kicadlib:TEST_0.100" H 4700 6150 60  0001 C CNN
 F 3 "" H 4700 6150 60  0000 C CNN
@@
 NoConn ~ 7550 2250
 NoConn ~ 7550 2400
-NoConn ~ 7550 2550
 Text Label 6900 4750 2    60   ~ 0
 batt+
@@
 P 4900 6150
 F 0 "P1" H 4900 6450 40  0000 C CNN
-F 1 "gnd" H 4900 6400 30  0000 C CNN
+F 1 "g" H 4900 6400 30  0000 C CNN
 F 2 "kicadlib:TEST_0.100" H 4900 6150 60  0001 C CNN
 F 3 "" H 4900 6150 60  0000 C CNN
@@
 P 6000 6150
 F 0 "P16" H 6000 6450 40  0000 C CNN
-F 1 "gnd" H 6000 6400 30  0000 C CNN
+F 1 "g" H 6000 6400 30  0000 C CNN
 F 2 "kicadlib:TEST_0.100" H 6000 6150 60  0001 C CNN
 F 3 "" H 6000 6150 60  0000 C CNN
@@
 Wire Wire Line
 	4900 6250 4900 6150
+Text Label 7650 2550 0    60   ~ 0
+mps_en
+Wire Wire Line
+	7650 2550 7550 2550
 $EndSCHEMATC
