File: hw/kicad/bttoy.kicad_pcb (KiCad board)
At the start: 2 copper layers, 45 parts, among them J1 USB-micro-b, J2 HC-07_BLUETOOTH, J3 ARM_10PIN, P1 +9V, P10 M1+, P11 M1-, P12 M2+, P13 M2-, P14 B-, P15 B+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

Commit message: place test points
Parts:
- added P16: g, kicadlib:TEST_0.100, F.Cu at (133.3, 72.4)
- P1: value +9V -> g
- P2: value i2c_sda -> sd
- P3: value i2c_scl -> sc
- P4: value spi_ss -> cs
- P5: value spi_miso -> mi
- P6: value spi_mosi -> mo
- P7: value spi_clk -> ck
- moved P8 68.0 mm to (165.1, 97.8)
- moved P9 63.9 mm to (165.1, 100.3)
- moved P2 42.1 mm to (125.7, 69.8)
- moved P4 38.4 mm to (130.8, 72.4)
- moved P1 38.1 mm to (128.3, 69.8)
- moved P3 38.0 mm to (123.2, 69.8)
- moved P5 37.7 mm to (125.7, 72.4)
- moved P7 33.3 mm to (128.3, 72.4)
- moved P6 24.7 mm to (123.2, 72.4)
- moved P10 23.4 mm to (123.2, 80.0)
- moved P11 22.7 mm to (123.2, 85.1)
- moved P15 8.76 mm to (134.6, 105.4)
- moved P13 8.52 mm to (166.4, 85.1)
- moved P14 8.52 mm to (137.2, 105.4)
- moved P12 8.24 mm to (166.4, 80.0)
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Connections:
- P1 pad 1: /+9V -> GND
Changed lines of the file:
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@@
-(kicad_pcb (version 4) (host pcbnew "(2014-10-27 BZR 5228)-product")
+(kicad_pcb (version 4) (host pcbnew "(after 2015-may-25 BZR unknown)-product")
   (general
-    (links 88)
-    (no_connects 88)
+    (links 89)
+    (no_connects 89)
     (area 0 0 0 0)
     (thickness 1.6)
-    (drawings 0)
+    (drawings 9)
     (tracks 0)
     (zones 0)
-    (modules 45)
+    (modules 46)
     (nets 85)
   )
@@
   )
   (module kicadlib:TEST_0.100 (layer F.Cu)
-    (at 121.92 107.442)
-    (fp_text reference P1 (at 0 -2.1) (layer F.SilkS) hide
-      (effects (font (size 1 1) (thickness 0.15)))
-    )
-    (fp_text value +9V (at 0 2.1) (layer F.SilkS)
-      (effects (font (size 1 1) (thickness 0.15)))
-    )
-    (pad 1 thru_hole circle (at 0 0) (size 1.75 1.75) (drill 1.02) (layers *.Cu *.Mask F.SilkS)
-      (net 3 /+9V))
-  )
-  (module kicadlib:TEST_0.100 (layer F.Cu)
-    (at 92.202 95.25)
+    (at 125.73 69.85)
     (fp_text reference P2 (at 0 -2.1) (layer F.SilkS) hide
       (effects (font (size 1 1) (thickness 0.15)))
     )
-    (fp_text value i2c_sda (at 0 2.1) (layer F.SilkS)
+    (fp_text value sd (at 0 4.318) (layer F.SilkS)
       (effects (font (size 1 1) (thickness 0.15)))
     )
@@
   )
   (module kicadlib:TEST_0.100 (layer F.Cu)
-    (at 89.408 87.249)
+    (at 123.19 69.85)
     (fp_text reference P3 (at 0 -2.1) (layer F.SilkS) hide
       (effects (font (size 1 1) (thickness 0.15)))
     )
-    (fp_text value i2c_scl (at 0 2.1) (layer F.SilkS)
+    (fp_text value sc (at 0 4.318) (layer F.SilkS)
       (effects (font (size 1 1) (thickness 0.15)))
     )
@@
   )
   (module kicadlib:TEST_0.100 (layer F.Cu)
-    (at 93.218 80.264)
+    (at 130.81 72.39)
     (fp_text reference P4 (at 0 -2.1) (layer F.SilkS) hide
       (effects (font (size 1 1) (thickness 0.15)))
     )
-    (fp_text value spi_ss (at 0 2.1) (layer F.SilkS)
+    (fp_text value cs (at 0 1.778) (layer F.SilkS)
       (effects (font (size 1 1) (thickness 0.15)))
     )
@@
   )
   (module kicadlib:TEST_0.100 (layer F.Cu)
-    (at 88.773 79.629)
+    (at 125.73 72.39)
     (fp_text reference P5 (at 0 -2.1) (layer F.SilkS) hide
       (effects (font (size 1 1) (thickness 0.15)))
     )
-    (fp_text value spi_miso (at 0 2.1) (layer F.SilkS)
+    (fp_text value mi (at 0 3.302) (layer F.SilkS)
       (effects (font (size 1 1) (thickness 0.15)))
     )
@@
   )
   (module kicadlib:TEST_0.100 (layer F.Cu)
-    (at 98.933 77.089)
+    (at 123.19 72.39)
     (fp_text reference P6 (at 0 -2.1) (layer F.SilkS) hide
       (effects (font (size 1 1) (thickness 0.15)))
     )
-    (fp_text value spi_mosi (at 0 2.1) (layer F.SilkS)
+    (fp_text value mo (at 0 3.302) (layer F.SilkS)
       (effects (font (size 1 1) (thickness 0.15)))
     )
@@
   )
   (module kicadlib:TEST_0.100 (layer F.Cu)
-    (at 101.854 92.71)
+    (at 128.27 72.39)
     (fp_text reference P7 (at 0 -2.1) (layer F.SilkS) hide
       (effects (font (size 1 1) (thickness 0.15)))
     )
-    (fp_text value spi_clk (at 0 2.1) (layer F.SilkS)
+    (fp_text value ck (at 0 3.302) (layer F.SilkS)
       (effects (font (size 1 1) (thickness 0.15)))
     )
@@
   )
   (module kicadlib:TEST_0.100 (layer F.Cu)
-    (at 98.298 85.344)
+    (at 165.1 97.79)
     (fp_text reference P8 (at 0 -2.1) (layer F.SilkS) hide
       (effects (font (size 1 1) (thickness 0.15)))
     )
-    (fp_text value +3.3v (at 0 2.1) (layer F.SilkS)
+    (fp_text value +3.3v (at -3.175 0) (layer F.SilkS)
       (effects (font (size 1 1) (thickness 0.15)))
     )
@@
   )
   (module kicadlib:TEST_0.100 (layer F.Cu)
-    (at 103.124 84.582)
+    (at 165.1 100.33)
     (fp_text reference P9 (at 0 -2.1) (layer F.SilkS) hide
       (effects (font (size 1 1) (thickness 0.15)))
     )
-    (fp_text value gnd (at 0 2.1) (layer F.SilkS)
-      (effects (font (size 1 1) (thickness 0.15)))
-    )
-    (pad 1 thru_hole circle (at 0 0) (size 1.75 1.75) (drill 1.02) (layers *.Cu *.Mask F.SilkS)
-      (net 2 GND))
-  )
-  (module kicadlib:TEST_0.100 (layer F.Cu)
-    (at 112.014 100.584)
+    (fp_text value gnd (at -2.54 0) (layer F.SilkS)
+      (effects (font (size 1 1) (thickness 0.15)))
+    )
+    (pad 1 thru_hole circle (at 0 0) (size 1.75 1.75) (drill 1.02) (layers *.Cu *.Mask F.SilkS)
+      (net 2 GND))
+  )
+  (module kicadlib:TEST_0.100 (layer F.Cu)
+    (at 123.19 80.01)
     (fp_text reference P10 (at 0 -2.1) (layer F.SilkS) hide
       (effects (font (size 1 1) (thickness 0.15)))
@@
   )
   (module kicadlib:TEST_0.100 (layer F.Cu)
-    (at 111.981666 104.879)
+    (at 123.19 85.09)
     (fp_text reference P11 (at 0 -2.1) (layer F.SilkS) hide
       (effects (font (size 1 1) (thickness 0.15)))
@@
   )
   (module kicadlib:TEST_0.100 (layer F.Cu)
-    (at 169.164 87.757)
+    (at 166.37 80.01)
     (fp_text reference P12 (at 0 -2.1) (layer F.SilkS) hide
       (effects (font (size 1 1) (thickness 0.15)))
@@
   )
   (module kicadlib:TEST_0.100 (layer F.Cu)
-    (at 168.91 93.218)
+    (at 166.37 85.09)
     (fp_text reference P13 (at 0 -2.1) (layer F.SilkS) hide
       (effects (font (size 1 1) (thickness 0.15)))
@@
   )
   (module kicadlib:TH_APEM_MHSS1105_SPDT (layer F.Cu)
-    (at 125.984 105.156)
+    (at 124.46 104.14)
     (fp_text reference SW1 (at 2.794 -1.778) (layer F.SilkS)
       (effects (font (size 0.75 0.75) (thickness 0.12)))
@@
   )
   (module kicadlib:TEST_0.100 (layer F.Cu)
-    (at 134.62 113.538)
+    (at 137.16 105.41)
     (fp_text reference P14 (at 0 -2.1) (layer F.SilkS) hide
       (effects (font (size 1 1) (thickness 0.15)))
     )
-    (fp_text value B- (at 0 2.1) (layer F.SilkS)
-      (effects (font (size 1 1) (thickness 0.15)))
-    )
-    (pad 1 thru_hole circle (at 0 0) (size 1.75 1.75) (drill 1.02) (layers *.Cu *.Mask F.SilkS)
-      (net 2 GND))
-  )
-  (module kicadlib:TEST_0.100 (layer F.Cu)
-    (at 131.064 113.411)
+    (fp_text value B- (at 2.286 0.254) (layer F.SilkS)
+      (effects (font (size 1 1) (thickness 0.15)))
+    )
+    (pad 1 thru_hole circle (at 0 0) (size 1.75 1.75) (drill 1.02) (layers *.Cu *.Mask F.SilkS)
+      (net 2 GND))
+  )
+  (module kicadlib:TEST_0.100 (layer F.Cu)
+    (at 134.62 105.41)
     (fp_text reference P15 (at 0 -2.1) (layer F.SilkS) hide
       (effects (font (size 1 1) (thickness 0.15)))
     )
-    (fp_text value B+ (at 0 2.1) (layer F.SilkS)
+    (fp_text value B+ (at -2.032 0) (layer F.SilkS)
       (effects (font (size 1 1) (thickness 0.15)))
     )
@@
       (net 1 /batt+))
   )
+  (module kicadlib:TEST_0.100 (layer F.Cu)
+    (at 128.27 69.85)
+    (fp_text reference P1 (at 0 -2.1) (layer F.SilkS) hide
+      (effects (font (size 1 1) (thickness 0.15)))
+    )
+    (fp_text value g (at 0 4.318) (layer F.SilkS)
+      (effects (font (size 1 1) (thickness 0.15)))
+    )
+    (pad 1 thru_hole circle (at 0 0) (size 1.75 1.75) (drill 1.02) (layers *.Cu *.Mask F.SilkS)
+      (net 2 GND))
+  )
+  (module kicadlib:TEST_0.100 (layer F.Cu)
+    (at 133.35 72.39)
+    (fp_text reference P16 (at 0 -2.1) (layer F.SilkS) hide
+      (effects (font (size 1 1) (thickness 0.15)))
+    )
+    (fp_text value g (at 0 1.778) (layer F.SilkS)
+      (effects (font (size 1 1) (thickness 0.15)))
+    )
+    (pad 1 thru_hole circle (at 0 0) (size 1.75 1.75) (drill 1.02) (layers *.Cu *.Mask F.SilkS)
+      (net 2 GND))
+  )
+  (gr_line (start 134.62 71.12) (end 129.54 71.12) (angle 90) (layer F.SilkS) (width 0.2))
+  (gr_line (start 134.62 73.66) (end 134.62 71.12) (angle 90) (layer F.SilkS) (width 0.2))
+  (gr_line (start 126.746 73.66) (end 134.62 73.66) (angle 90) (layer F.SilkS) (width 0.2))
+  (gr_line (start 121.92 73.66) (end 125.984 73.66) (angle 90) (layer F.SilkS) (width 0.2))
+  (gr_line (start 121.92 71.12) (end 121.92 73.66) (angle 90) (layer F.SilkS) (width 0.2))
+  (gr_line (start 121.92 71.12) (end 121.92 68.58) (angle 90) (layer F.SilkS) (width 0.2))
+  (gr_line (start 129.54 71.12) (end 121.92 71.12) (angle 90) (layer F.SilkS) (width 0.2))
+  (gr_line (start 129.54 68.58) (end 129.54 71.12) (angle 90) (layer F.SilkS) (width 0.2))
+  (gr_line (start 121.92 68.58) (end 129.54 68.58) (angle 90) (layer F.SilkS) (width 0.2))
 )

Commit message: gerbers and done
Parts:
- moved P10 43.2 mm to (166.4, 80.0)
- moved P11 43.2 mm to (166.4, 85.1)
- moved P12 43.2 mm to (123.2, 80.0)
- moved P13 43.2 mm to (123.2, 85.1)
- moved P4 7.62 mm to (123.2, 72.4)
- moved P6 5.08 mm to (128.3, 72.4)
- moved P2 2.54 mm to (123.2, 69.8)
- moved P3 2.54 mm to (125.7, 69.8)
- moved P7 2.54 mm to (130.8, 72.4)
Connections:
- U4 pad 10: /acc_spi_miso -> /spi_miso
- U4 pad 17: Net-(U4-Pad17) -> /mps_en
Routing:
- net /+3.3v: track 0.00 -> 69.5 mm, vias 0 -> 2
- net /vbatt_out: track 0.00 -> 59.4 mm, vias 0 -> 2
- net /motor_1_+: track 0.00 -> 32.7 mm, vias 0 -> 1
- net /motor_1_-: track 0.00 -> 31.2 mm, vias 0 -> 1
- net /mps_en: track 0.00 -> 27.7 mm
- net GND: track 0.00 -> 27.4 mm, vias 0 -> 6
- net /motor_2_+: track 0.00 -> 25.1 mm, vias 0 -> 1
- net /i2c_sda: track 0.00 -> 24.0 mm, vias 0 -> 1
- net /spi_ss: track 0.00 -> 23.3 mm, vias 0 -> 2
- net /batt+: track 0.00 -> 22.6 mm
- net /motor_2_-: track 0.00 -> 22.0 mm, vias 0 -> 1
- net /spi_mosi: track 0.00 -> 21.9 mm, vias 0 -> 1
- net /i2c_scl: track 0.00 -> 21.7 mm, vias 0 -> 1
- net /spi_miso: track 0.00 -> 20.8 mm, vias 0 -> 1
- net /spi_sclk: track 0.00 -> 20.7 mm, vias 0 -> 1
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- added copper zone on B.Cu, net GND
- added copper zone on F.Cu, net GND
Other:
- board outline added: 48.3 x 40.6 mm
- net class pwr added: clearance 0.254, trace_width 0.4, via_dia 0.889, via_drill 0.635
- board text added: "github.com/noahp/bttoy v0.1 Sept 2015"
